File: Design/H14R90.sch (EAGLE design)
At the start: 39 parts, among them P2 HEXABIT_17.32_NO_P6, Q1 MMBT3904LT1, Q2 MMBT3904LT1, Q3 MMBT3904LT1, Q4 MMBT3904LT1, U1 STM32G0B1CEU6N, U2 LM2775-Q1, X1 XTALL_CSTCE8M00G52

Commit message: -Correcting some documentaion issues
Other:
- note added: "H14R9"
- note added: "H14R9_Backend"
- note added: "H14R9_Frontend"
- note removed: "H14R90"
- note removed: "H14R90_Backend"
- note removed: "H14R90_Frontend"
Changed lines of the file:
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@@
 <?xml version="1.0" encoding="utf-8"?>
 <!DOCTYPE eagle SYSTEM "eagle.dtd">
-<eagle version="9.6.1">
+<eagle version="9.6.2">
 <drawing>
 <settings>
@@
 <text x="216.45" y="4.9548" size="1.9304" layer="100" font="vector">Sheet   of</text>
 <text x="200.0162" y="19.2042" size="1.9304" layer="100" font="vector">Title</text>
-<text x="181.4742" y="19.2042" size="1.9304" layer="102" font="vector">H14R90</text>
+<text x="181.4742" y="19.2042" size="1.9304" layer="102" font="vector">H14R9</text>
 <text x="186.7828" y="11.4064" size="1.9304" layer="101" font="vector">4 x 5V PWM O/P
 + External Supply </text>
-<text x="206.8742" y="19.2042" size="1.9304" layer="101" font="vector">H14R90_Backend</text>
+<text x="206.8742" y="19.2042" size="1.9304" layer="101" font="vector">H14R9_Backend</text>
 <wire x1="169.46" y1="3.38" x2="169.46" y2="7.698" width="0.1524" layer="205"/>
 <wire x1="169.46" y1="7.698" x2="169.46" y2="17.858" width="0.1524" layer="205"/>
@@
 <text x="216.45" y="4.9548" size="1.9304" layer="100" font="vector">Sheet   of</text>
 <text x="200.0162" y="19.2042" size="1.9304" layer="100" font="vector">Title</text>
-<text x="181.4742" y="19.2042" size="1.9304" layer="102" font="vector">H14R90</text>
+<text x="181.4742" y="19.2042" size="1.9304" layer="102" font="vector">H14R9</text>
 <text x="188.0528" y="11.4064" size="1.9304" layer="101" font="vector">4 x 5V PWM O/P
 + External Supply </text>
-<text x="206.8742" y="19.2042" size="1.9304" layer="101" font="vector">H14R90_Frontend</text>
+<text x="206.8742" y="19.2042" size="1.9304" layer="101" font="vector">H14R9_Frontend</text>
 <wire x1="169.46" y1="3.38" x2="169.46" y2="7.698" width="0.1524" layer="205"/>
 <wire x1="169.46" y1="7.698" x2="169.46" y2="17.858" width="0.1524" layer="205"/>
